Commit message: fixed the wheel. The issue was the axis of the pitch due to inertia

File: src/gnc_description/urdf/Base.urdf.xacro (robot description, xacro)
@@ -2,6 +2,6 @@
 <robot xmlns:xacro="http://www.ros.org/wiki/xacro" name="base">
     <!-- This is values for the base of the robot -->
-    <xacro:property name="baseLength" value="0.4" />
-    <xacro:property name="baseWidth" value="0.5" />
+    <xacro:property name="baseLength" value="0.5" />
+    <xacro:property name="baseWidth" value="0.4" />
     <xacro:property name="baseHeight" value="0.1" />
     <xacro:property name="originBaseX" value="0" />

File: src/gnc_description/urdf/Wheel.urdf.xacro (robot description, xacro)
@@ -11,5 +11,5 @@
         <link name="${name}_link">
             <visual>
-                <origin xyz="${originWheelX} ${originWheelY} ${originWheelZ}" rpy="0 ${pi/2} 0"/>
+                <origin xyz="${originWheelX} ${originWheelY} ${originWheelZ}" rpy="${pi/2} 0 0"/>
                 <geometry>
                     <cylinder length="${wheelLength}" radius="${wheelRadius}"/>
@@ -18,5 +18,5 @@
             </visual>
             <collision>
-                <origin xyz="${originWheelX} ${originWheelY} ${originWheelZ}" rpy="0 ${pi/2} 0"/>
+                <origin xyz="${originWheelX} ${originWheelY} ${originWheelZ}" rpy="${pi/2} 0 0"/>
                 <geometry>
                     <cylinder length="${wheelLength}" radius="${wheelRadius}"/>
@@ -31,5 +31,5 @@
         </link>
         <joint name="${name}_joint" type="continuous">
-            <origin xyz="${WheelXOrigin} ${WheelYOrigin} 0" rpy="0 0 0"/>
+            <origin xyz="${WheelXOrigin} ${WheelYOrigin} 0" rpy="0 ${pi/2} 0"/>
             <parent link="${parentLink}"/>
             <child link="${name}_link"/>

File: src/gnc_description/urdf/protobot.urdf.xacro (robot description, xacro)
@@ -16,11 +16,11 @@
     <xacro:base name="base" mass="${baseMass}"/>
     <!-- Left Side of the wheels -->
-    <xacro:wheel name="wheel_Left_Front"  mass="${wheelMass}" parentLink="base_link" WheelXOrigin="${LeftWheelXOrigin}" WheelYOrigin="${FrontWheelYOrigin}"/>
-    <xacro:wheel name="wheel_Left_Middle" mass="${wheelMass}" parentLink="base_link" WheelXOrigin="${LeftWheelXOrigin}" WheelYOrigin="${MiddleWheelYOrigin}"/>
-    <xacro:wheel name="wheel_Left_Back" mass="${wheelMass}" parentLink="base_link" WheelXOrigin="${LeftWheelXOrigin}" WheelYOrigin="${BackWheelYOrigin}"/>
+    <xacro:wheel name="wheel_Left_Front"  mass="${wheelMass}" parentLink="base_link" WheelXOrigin="${FrontWheelYOrigin}" WheelYOrigin="${LeftWheelXOrigin}"/>
+    <xacro:wheel name="wheel_Left_Middle" mass="${wheelMass}" parentLink="base_link" WheelXOrigin="${MiddleWheelYOrigin}" WheelYOrigin="${LeftWheelXOrigin}"/>
+    <xacro:wheel name="wheel_Left_Back" mass="${wheelMass}" parentLink="base_link" WheelXOrigin="${BackWheelYOrigin}" WheelYOrigin="${LeftWheelXOrigin}"/>
     <!-- Right Side of the wheels -->
-    <xacro:wheel name="wheel_Right_Front" mass="${wheelMass}" parentLink="base_link" WheelXOrigin="${RightWheelXOrigin}" WheelYOrigin="${FrontWheelYOrigin}"/>
-    <xacro:wheel name="wheel_Right_Middle" mass="${wheelMass}" parentLink="base_link" WheelXOrigin="${RightWheelXOrigin}" WheelYOrigin="${MiddleWheelYOrigin}"/>
-    <xacro:wheel name="wheel_Right_Back" mass="${wheelMass}" parentLink="base_link" WheelXOrigin="${RightWheelXOrigin}" WheelYOrigin="${BackWheelYOrigin}"/>
+    <xacro:wheel name="wheel_Right_Front" mass="${wheelMass}" parentLink="base_link" WheelXOrigin="${FrontWheelYOrigin}" WheelYOrigin="${RightWheelXOrigin}"/>
+    <xacro:wheel name="wheel_Right_Middle" mass="${wheelMass}" parentLink="base_link" WheelXOrigin="${MiddleWheelYOrigin}" WheelYOrigin="${RightWheelXOrigin}"/>
+    <xacro:wheel name="wheel_Right_Back" mass="${wheelMass}" parentLink="base_link" WheelXOrigin="${BackWheelYOrigin}" WheelYOrigin="${RightWheelXOrigin}"/>
     <!-- Gazebo code for protobot -->
     <gazebo>
