Commit message: Delete not needed files and folders and reorganized

File: src/gnc_description/urdf/_T265.xacro (robot description, xacro)
@@ -92,5 +92,5 @@
             <origin rpy="1.57 0 1.57" xyz="0 0 0"/>
             <geometry>
-                <mesh filename="package://realsense2_description/meshes/realsense_t265.stl" scale="0.001 0.001 0.001"/>
+                <mesh filename="package://gnc_description/meshes/realsense_t265.stl" scale="0.001 0.001 0.001"/>
             </geometry>
         </visual>

File: src/gnc_description/urdf/_d435i.xacro (robot description, xacro)
@@ -44,5 +44,5 @@
         <origin xyz="${d435_cam_mount_from_center_offset} ${-d435_cam_depth_py} 0" rpy="${pi/2} 0 ${pi/2}"/>
         <geometry>
-          <mesh filename="package://realsense2_description/meshes/d435.dae" />
+          <mesh filename="package://gnc_description/meshes/d435.dae" />
         </geometry>
       </visual>

File: src/gnc_description/urdf/gnc_robot.xacro (robot description, xacro)
@@ -24,6 +24,6 @@
     <xacro:wheel name="wheel_Right_Back" mass="${wheelMass}" parentLink="base_link" WheelXOrigin="${BackWheelYOrigin}" WheelYOrigin="${RightWheelXOrigin}"/>
     <!-- Camera -->
-    <xacro:include filename="$(find realsense2_description)/urdf/_d435i.urdf.xacro" />
-    <xacro:include filename="$(find realsense2_description)/urdf/_T265.urdf.xacro"/>
+    <xacro:include filename="_d435i.xacro" />
+    <xacro:include filename="_T265.xacro"/>
     <xacro:arg name="use_nominal_extrinsics" default="True" />
     <xacro:realsense_d435 sensor_name="camera" parent_link="base_link" rate="30.0">
