Commit message: Finish the cameras for URDF

File: src/gnc_description/urdf/Wheel.xacro (robot description, xacro)
@@ -3,5 +3,5 @@
     <!-- This is values for the Wheels of the robot -->
     <xacro:property name="wheelLength" value="0.05" />
-    <xacro:property name="wheelRadius" value="0.09" />
+    <xacro:property name="wheelRadius" value="0.1" />
     <xacro:property name="originWheelX" value="0"/>
     <xacro:property name="originWheelY" value="0"/>

File: src/gnc_description/urdf/gnc_robot.xacro (robot description, xacro)
@@ -23,4 +23,14 @@
     <xacro:wheel name="wheel_Right_Middle" mass="${wheelMass}" parentLink="base_link" WheelXOrigin="${MiddleWheelYOrigin}" WheelYOrigin="${RightWheelXOrigin}"/>
     <xacro:wheel name="wheel_Right_Back" mass="${wheelMass}" parentLink="base_link" WheelXOrigin="${BackWheelYOrigin}" WheelYOrigin="${RightWheelXOrigin}"/>
+    <!-- Camera -->
+    <xacro:include filename="$(find realsense2_description)/urdf/_d435i.urdf.xacro" />
+    <xacro:include filename="$(find realsense2_description)/urdf/_T265.urdf.xacro"/>
+    <xacro:arg name="use_nominal_extrinsics" default="True" />
+    <xacro:realsense_d435 sensor_name="camera" parent_link="base_link" rate="30.0">
+        <origin xyz="0.20 0 0.15" rpy="0 0 0"/>
+    </xacro:realsense_d435>
+    <xacro:realsense_T265 sensor_name="camera_z" parent_link="base_link" rate="30.0">
+        <origin rpy="0 0 0" xyz="0 0 0.25"/>
+    </xacro:realsense_T265>
     <!-- Gazebo code for protobot -->
     <gazebo>

Commit message: changed wheel mesh and tweaked values

File: src/gnc_description/urdf/Wheel.xacro (robot description, xacro)
@@ -11,5 +11,5 @@
         <link name="${name}_link">
             <visual>
-                <origin xyz="${originWheelX} ${originWheelY} ${originWheelZ}" rpy="0 0 ${pi/2}"/>
+                <origin xyz="${originWheelX} ${originWheelY} ${originWheelZ}" rpy="0 0 0"/>
                 <geometry>
                     <mesh filename="package://gnc_gazebo/mesh/wheel.stl"/>

File: src/gnc_description/urdf/gnc_robot.xacro (robot description, xacro)
@@ -16,11 +16,11 @@
     <xacro:base name="base" mass="${baseMass}"/>
     <!-- Left Side of the wheels -->
-    <xacro:wheel name="wheel_Left_Front"  mass="${wheelMass}" parentLink="base_link" WheelXOrigin="${FrontWheelYOrigin}" WheelYOrigin="${LeftWheelXOrigin}"/>
-    <xacro:wheel name="wheel_Left_Middle" mass="${wheelMass}" parentLink="base_link" WheelXOrigin="${MiddleWheelYOrigin}" WheelYOrigin="${LeftWheelXOrigin}"/>
-    <xacro:wheel name="wheel_Left_Back" mass="${wheelMass}" parentLink="base_link" WheelXOrigin="${BackWheelYOrigin}" WheelYOrigin="${LeftWheelXOrigin}"/>
+    <xacro:wheel name="wheel_Right_Front"  mass="${wheelMass}" parentLink="base_link" WheelXOrigin="${FrontWheelYOrigin}" WheelYOrigin="${LeftWheelXOrigin}"/>
+    <xacro:wheel name="wheel_Right_Middle" mass="${wheelMass}" parentLink="base_link" WheelXOrigin="${MiddleWheelYOrigin}" WheelYOrigin="${LeftWheelXOrigin}"/>
+    <xacro:wheel name="wheel_Right_Back" mass="${wheelMass}" parentLink="base_link" WheelXOrigin="${BackWheelYOrigin}" WheelYOrigin="${LeftWheelXOrigin}"/>
     <!-- Right Side of the wheels -->
-    <xacro:wheel name="wheel_Right_Front" mass="${wheelMass}" parentLink="base_link" WheelXOrigin="${FrontWheelYOrigin}" WheelYOrigin="${RightWheelXOrigin}"/>
-    <xacro:wheel name="wheel_Right_Middle" mass="${wheelMass}" parentLink="base_link" WheelXOrigin="${MiddleWheelYOrigin}" WheelYOrigin="${RightWheelXOrigin}"/>
-    <xacro:wheel name="wheel_Right_Back" mass="${wheelMass}" parentLink="base_link" WheelXOrigin="${BackWheelYOrigin}" WheelYOrigin="${RightWheelXOrigin}"/>
+    <xacro:wheel name="wheel_Left_Front" mass="${wheelMass}" parentLink="base_link" WheelXOrigin="${FrontWheelYOrigin}" WheelYOrigin="${RightWheelXOrigin}"/>
+    <xacro:wheel name="wheel_Left_Middle" mass="${wheelMass}" parentLink="base_link" WheelXOrigin="${MiddleWheelYOrigin}" WheelYOrigin="${RightWheelXOrigin}"/>
+    <xacro:wheel name="wheel_Left_Back" mass="${wheelMass}" parentLink="base_link" WheelXOrigin="${BackWheelYOrigin}" WheelYOrigin="${RightWheelXOrigin}"/>
     <!-- Camera -->
     <xacro:include filename="_d435i.xacro" />
