Commit message: Work

File: src/gnc_description/urdf/gnc_robot_backup.xacro (robot description, xacro)
@@ -34,8 +34,9 @@
     </xacro:realsense_T265>
     <!-- IMU GPS -->
-    <xacro:include filename="$(find gnc_gazebo)/sensors/_zedf9r.xacro"/>
-    <xacro:Sparkfun_zedf9r name="zed_Sensor" parentLink="base_link">
-       <origin rpy="0 0 0" xyz="0 0 0.15"/>
-    </xacro:Sparkfun_zedf9r>
+    <!--    <xacro:include filename="$(find gnc_gazebo)/sensors/_zedf9r.xacro"/>
+        <xacro:Sparkfun_zedf9r name="zed_Sensor" parentLink="base_link">
+            <origin rpy="0 0 0" xyz="0 0 0.15"/>
+        </xacro:Sparkfun_zedf9r>
+	-->
     <!-- Gazebo code for protobot -->
     <gazebo>

File: src/gnc_gazebo/sensors/_zedf9r.xacro (robot description, xacro)
@@ -1,4 +1,4 @@
 <?xml version="1.0"?>
-<robot xmlns:xacro="http://www.ros.org/wiki/xacro" name="sensor_zedf9r">
+<robot xmlns:xacro="http://www.ros.org/wiki/xacro" name="zed_Sensor">
     <xacro:property name="baseZedLength" value="0.0508" />
     <xacro:property name="baseZedWidth" value="0.04318" />
@@ -40,5 +40,5 @@
                 <topicName>gps/fix</topicName>
                 <frameId>${name}_link</frameId>
-                <gaussianNoise>0</gaussianNoise>
+                <gaussianNoise>2</gaussianNoise>
                 <alwayson>true</alwayson>
             </plugin>
@@ -48,5 +48,5 @@
                 <topicName>imu/data</topicName>
                 <serviceName>imu_service</serviceName>
-                <gaussianNoise>0</gaussianNoise>
+                <gaussianNoise>0.1</gaussianNoise>
                 <updateRate>30.0</updateRate>
             </plugin>
