Commit message: updated urdf, collision sizes and joint locations, added meshes

File: src/gnc_description/urdf/Base.xacro (robot description, xacro)
@@ -2,7 +2,7 @@
 <robot xmlns:xacro="http://www.ros.org/wiki/xacro" name="base">
     <!-- This is values for the base of the robot -->
-    <xacro:property name="baseLength" value="0.5" />
-    <xacro:property name="baseWidth" value="0.4" />
-    <xacro:property name="baseHeight" value="0.1" />
+    <xacro:property name="baseLength" value="0.86" />
+    <xacro:property name="baseWidth" value="0.67" />
+    <xacro:property name="baseHeight" value="0.53" />
     <xacro:property name="originBaseX" value="0" />
     <xacro:property name="originBaseY" value="0" />
@@ -14,7 +14,6 @@
                 <origin xyz="${originBaseX} ${originBaseY} ${originBaseZ}" rpy="0 0 0"/>
                 <geometry>
-                    <box size="${baseLength} ${baseWidth} ${baseHeight}" />
+                    <mesh filename="package://gnc_gazebo/mesh/chassis.stl"/>
                 </geometry>
-                <material name="${baseColor}"/>
             </visual>
             <collision>

File: src/gnc_description/urdf/Wheel.xacro (robot description, xacro)
@@ -2,6 +2,6 @@
 <robot xmlns:xacro="http://www.ros.org/wiki/xacro" name="wheel">
     <!-- This is values for the Wheels of the robot -->
-    <xacro:property name="wheelLength" value="0.05" />
-    <xacro:property name="wheelRadius" value="0.1" />
+    <xacro:property name="wheelLength" value="0.1016" />
+    <xacro:property name="wheelRadius" value="0.09" />
     <xacro:property name="originWheelX" value="0"/>
     <xacro:property name="originWheelY" value="0"/>
@@ -11,9 +11,8 @@
         <link name="${name}_link">
             <visual>
-                <origin xyz="${originWheelX} ${originWheelY} ${originWheelZ}" rpy="${pi/2} 0 0"/>
+                <origin xyz="${originWheelX} ${originWheelY} ${originWheelZ}" rpy="0 0 ${pi/2}"/>
                 <geometry>
-                    <cylinder length="${wheelLength}" radius="${wheelRadius}"/>
+                    <mesh filename="package://gnc_gazebo/mesh/wheel.stl"/>
                 </geometry>
-                <material name="${wheelColor}"/>
             </visual>
             <collision>
@@ -31,5 +30,5 @@
         </link>
         <joint name="${name}_joint" type="continuous">
-            <origin xyz="${WheelXOrigin} ${WheelYOrigin} 0" rpy="0 ${pi/2} 0"/>
+            <origin xyz="${WheelXOrigin} ${WheelYOrigin} -0.27" rpy="0 ${pi/2} 0"/>
             <parent link="${parentLink}"/>
             <child link="${name}_link"/>

File: src/gnc_description/urdf/gnc_robot.xacro (robot description, xacro)
@@ -6,11 +6,11 @@
     <xacro:include filename="material.xacro" />
     <!-- Wheel Origin Values -->
-    <xacro:property name="LeftWheelXOrigin" value="-.23"/>
-    <xacro:property name="RightWheelXOrigin" value=".23"/>
-    <xacro:property name="BackWheelYOrigin" value="-.2"/>
+    <xacro:property name="LeftWheelXOrigin" value="-.32"/>
+    <xacro:property name="RightWheelXOrigin" value=".32"/>
+    <xacro:property name="BackWheelYOrigin" value="-.38"/>
     <xacro:property name="MiddleWheelYOrigin" value="0"/>
-    <xacro:property name="FrontWheelYOrigin" value=".2"/>
-    <xacro:property name="wheelMass" value="1"/>
-    <xacro:property name="baseMass" value="1"/>
+    <xacro:property name="FrontWheelYOrigin" value=".38"/>
+    <xacro:property name="wheelMass" value="0.7"/>
+    <xacro:property name="baseMass" value="20"/>
     <!-- Base of the robot -->
     <xacro:base name="base" mass="${baseMass}"/>

Commit message: Work

File: src/gnc_description/urdf/Base.xacro (robot description, xacro)
@@ -14,5 +14,5 @@
                 <origin xyz="${originBaseX} ${originBaseY} ${originBaseZ}" rpy="0 0 0"/>
                 <geometry>
-                    <mesh filename="package://gnc_gazebo/mesh/chassis.stl"/>
+                    <mesh filename="package://gnc_description/mesh/chassis.stl"/>
                 </geometry>
             </visual>

File: src/gnc_description/urdf/Wheel.xacro (robot description, xacro)
@@ -13,5 +13,5 @@
                 <origin xyz="${originWheelX} ${originWheelY} ${originWheelZ}" rpy="0 0 0"/>
                 <geometry>
-                    <mesh filename="package://gnc_gazebo/mesh/wheel.stl"/>
+                    <mesh filename="package://gnc_description/mesh/wheel.dae"/>
                 </geometry>
             </visual>

File: src/gnc_description/urdf/gnc_robot.xacro (robot description, xacro)
@@ -9,5 +9,4 @@
     <xacro:property name="RightWheelXOrigin" value=".32"/>
     <xacro:property name="BackWheelYOrigin" value="-.38"/>
-    <xacro:property name="MiddleWheelYOrigin" value="0"/>
     <xacro:property name="FrontWheelYOrigin" value=".38"/>
     <xacro:property name="wheelMass" value="0.7"/>
@@ -17,9 +16,7 @@
     <!-- Left Side of the wheels -->
     <xacro:wheel name="wheel_Right_Front"  mass="${wheelMass}" parentLink="base_link" WheelXOrigin="${FrontWheelYOrigin}" WheelYOrigin="${LeftWheelXOrigin}"/>
-    <xacro:wheel name="wheel_Right_Middle" mass="${wheelMass}" parentLink="base_link" WheelXOrigin="${MiddleWheelYOrigin}" WheelYOrigin="${LeftWheelXOrigin}"/>
     <xacro:wheel name="wheel_Right_Back" mass="${wheelMass}" parentLink="base_link" WheelXOrigin="${BackWheelYOrigin}" WheelYOrigin="${LeftWheelXOrigin}"/>
     <!-- Right Side of the wheels -->
     <xacro:wheel name="wheel_Left_Front" mass="${wheelMass}" parentLink="base_link" WheelXOrigin="${FrontWheelYOrigin}" WheelYOrigin="${RightWheelXOrigin}"/>
-    <xacro:wheel name="wheel_Left_Middle" mass="${wheelMass}" parentLink="base_link" WheelXOrigin="${MiddleWheelYOrigin}" WheelYOrigin="${RightWheelXOrigin}"/>
     <xacro:wheel name="wheel_Left_Back" mass="${wheelMass}" parentLink="base_link" WheelXOrigin="${BackWheelYOrigin}" WheelYOrigin="${RightWheelXOrigin}"/>
     <!-- Camera -->
@@ -31,5 +28,5 @@
     <xacro:arg name="use_nominal_extrinsics" default="True" />
     <xacro:zed_camera name="ZEDMini" parent="base_link">
-        <origin xyz="0.20 0 0.1805" rpy="0 0 0"/>
+        <origin xyz="0.0 0 0" rpy="0 0 0"/>
     </xacro:zed_camera>
 <!--
@@ -57,8 +54,6 @@
             <update_rate>20</update_rate>
             <joint_name>wheel_Left_Front_joint</joint_name>
-            <joint_name>wheel_Left_Middle_joint</joint_name>
             <joint_name>wheel_Left_Back_joint</joint_name>
             <joint_name>wheel_Right_Front_joint</joint_name>
-            <joint_name>wheel_Right_Middle_joint</joint_name>
             <joint_name>wheel_Right_Back_joint</joint_name>
         </plugin>
@@ -76,17 +71,4 @@
     </joint>
     <link name="teleop_camera_link"/>
-    <joint name="arm_joint" type="fixed">
-        <origin xyz="-0.113 -0.0174 0.235" rpy="0 0 0"/>
-        <parent link="base_link"/>
-        <child link="arm_link"/>
-    </joint>
-    <link name="arm_link">
-        <visual>
-            <origin xyz="0 0 0" rpy="0 0 0"/>
-            <geometry>
-                <mesh filename="package://gnc_gazebo/mesh/arm.stl"/>
-            </geometry>
-        </visual>
-    </link>
     <link name="magnetometer"/>
     <gazebo>

File: src/gnc_gazebo/sensors/_ZED.xacro (robot description, xacro)
@@ -28,4 +28,5 @@
 		<parent link="${parent}"/>
 		<child link="${name}"/>
+		<origin xyz="0.6 0 0 " rpy="0 0 0 "/>
 	</joint>
 	<joint name="${name}_imu_joint" type="fixed">
@@ -35,5 +36,5 @@
 	<link name="${name}_optical_frame"/>
 	<joint name="${name}_optical_joint" type="fixed">
-		<parent link="${parent}"/>
+		<parent link="${name}"/>
 		<child link="${name}_optical_frame"/>
 		<origin xyz="0 0 0" rpy="1.5708 0 0"/>

Commit message: Work

File: src/gnc_description/urdf/Base.xacro (robot description, xacro)
@@ -2,6 +2,6 @@
 <robot xmlns:xacro="http://www.ros.org/wiki/xacro" name="base">
     <!-- This is values for the base of the robot -->
-    <xacro:property name="baseLength" value="0.86" />
-    <xacro:property name="baseWidth" value="0.67" />
+    <xacro:property name="baseLength" value="0.779" />
+    <xacro:property name="baseWidth" value="0.780" />
     <xacro:property name="baseHeight" value="0.53" />
     <xacro:property name="originBaseX" value="0" />

File: src/gnc_description/urdf/Wheel.xacro (robot description, xacro)
@@ -2,6 +2,6 @@
 <robot xmlns:xacro="http://www.ros.org/wiki/xacro" name="wheel">
     <!-- This is values for the Wheels of the robot -->
-    <xacro:property name="wheelLength" value="0.1016" />
-    <xacro:property name="wheelRadius" value="0.09" />
+    <xacro:property name="wheelLength" value="0.02" />
+    <xacro:property name="wheelRadius" value="0.08" />
     <xacro:property name="originWheelX" value="0"/>
     <xacro:property name="originWheelY" value="0"/>

File: src/gnc_description/urdf/gnc_robot.xacro (robot description, xacro)
@@ -6,8 +6,8 @@
     <xacro:include filename="material.xacro" />
     <!-- Wheel Origin Values -->
-    <xacro:property name="LeftWheelXOrigin" value="-.32"/>
-    <xacro:property name="RightWheelXOrigin" value=".32"/>
-    <xacro:property name="BackWheelYOrigin" value="-.38"/>
-    <xacro:property name="FrontWheelYOrigin" value=".38"/>
+    <xacro:property name="LeftWheelXOrigin" value="-.37"/>
+    <xacro:property name="RightWheelXOrigin" value=".37"/>
+    <xacro:property name="BackWheelYOrigin" value="-.37"/>
+    <xacro:property name="FrontWheelYOrigin" value=".37"/>
     <xacro:property name="wheelMass" value="0.7"/>
     <xacro:property name="baseMass" value="20"/>
