Commit message: Got the gps and imu finished for the zedf9r

File: src/gnc_description/urdf/gnc_robot.xacro (robot description, xacro)
@@ -24,6 +24,6 @@
     <xacro:wheel name="wheel_Right_Back" mass="${wheelMass}" parentLink="base_link" WheelXOrigin="${BackWheelYOrigin}" WheelYOrigin="${RightWheelXOrigin}"/>
     <!-- Camera -->
-    <xacro:include filename="_d435i.xacro" />
-    <xacro:include filename="_T265.xacro"/>
+    <xacro:include filename="sensors/_d435i.xacro" />
+    <xacro:include filename="sensors/_T265.xacro"/>
     <xacro:arg name="use_nominal_extrinsics" default="True" />
     <xacro:realsense_d435 sensor_name="camera" parent_link="base_link" rate="30.0">
@@ -33,4 +33,9 @@
         <origin rpy="0 0 0" xyz="0 0 0.25"/>
     </xacro:realsense_T265>
+    <!-- IMU GPS -->
+        <xacro:include filename="sensors/_zedf9r.xacro"/>
+        <xacro:Sparkfun_zedf9r name="zed_Sensor" parentLink="base_link">
+            <origin rpy="0 0 0" xyz="0 0 0.15"/>
+        </xacro:Sparkfun_zedf9r>
     <!-- Gazebo code for protobot -->
     <gazebo>

File: src/gnc_description/urdf/material.xacro (robot description, xacro)
@@ -7,3 +7,6 @@
         <color rgba="0 0 0 1"/>
     </material>
+    <material name="Red">
+        <color rgba="1 0 0 1"/>
+    </material>
 </robot>

Commit message: Updated iFiles

File: src/gnc_description/urdf/gnc_robot.xacro (robot description, xacro)
@@ -24,6 +24,6 @@
     <xacro:wheel name="wheel_Left_Back" mass="${wheelMass}" parentLink="base_link" WheelXOrigin="${BackWheelYOrigin}" WheelYOrigin="${RightWheelXOrigin}"/>
     <!-- Camera -->
-    <xacro:include filename="sensors/_d435i.xacro" />
-    <xacro:include filename="sensors/_T265.xacro"/>
+    <xacro:include filename="$(find gnc_gazebo)/sensors/_d435i.xacro" />
+    <xacro:include filename="$(find gnc_gazebo)/sensors/_T265.xacro"/>
     <xacro:arg name="use_nominal_extrinsics" default="True" />
     <xacro:realsense_d435 sensor_name="camera" parent_link="base_link" rate="30.0">
@@ -34,5 +34,5 @@
     </xacro:realsense_T265>
     <!-- IMU GPS -->
-        <xacro:include filename="sensors/_zedf9r.xacro"/>
+        <xacro:include filename="$(find gnc_gazebo)/sensors/_zedf9r.xacro"/>
         <xacro:Sparkfun_zedf9r name="zed_Sensor" parentLink="base_link">
             <origin rpy="0 0 0" xyz="0 0 0.15"/>

File: src/gnc_gazebo/sensors/_T265.xacro (robot description, xacro)
@@ -92,5 +92,5 @@
             <origin rpy="1.57 0 1.57" xyz="0 0 0"/>
             <geometry>
-                <mesh filename="package://gnc_description/meshes/realsense_t265.stl" scale="0.001 0.001 0.001"/>
+                <mesh filename="package://gnc_gazebo/meshes/realsense_t265.stl" scale="0.001 0.001 0.001"/>
             </geometry>
         </visual>

File: src/gnc_gazebo/sensors/_d435i.xacro (robot description, xacro)
@@ -44,5 +44,5 @@
         <origin xyz="${d435_cam_mount_from_center_offset} ${-d435_cam_depth_py} 0" rpy="${pi/2} 0 ${pi/2}"/>
         <geometry>
-          <mesh filename="package://gnc_description/meshes/d435.dae" />
+          <mesh filename="package://gnc_gazebo/meshes/d435.dae" />
         </geometry>
       </visual>

Commit message: arm addition

File: src/gnc_description/urdf/gnc_robot.xacro (robot description, xacro)
@@ -57,3 +57,61 @@
         </plugin>
     </gazebo>
+    <joint name="teleop_camera_joint" type="fixed">
+    <origin xyz="-0.181 0.19 0.695" rpy="0 0 0"/>
+    <parent link="base_link"/>
+    <child link="teleop_camera_link"/>
+    </joint>
+    <link name="teleop_camera_link"/>
+    <joint name="arm_joint" type="fixed">
+        <origin xyz="-0.113 -0.0174 0.235" rpy="0 0 0"/>
+        <parent link="base_link"/>
+        <child link="arm_link"/>
+    </joint>
+    <link name="arm_link">
+        <visual>
+            <origin xyz="0 0 0" rpy="0 0 0"/>
+            <geometry>
+                <mesh filename="package://gnc_gazebo/mesh/arm.stl"/>
+            </geometry>
+        </visual>
+    </link>
+    <gazebo reference="teleop_camera_link">
+    <sensor type="camera" name="teleop_cam">
+      <update_rate>30.0</update_rate>
+      <camera name="teleop_cam">
+        <horizontal_fov>1.3962634</horizontal_fov>
+        <image>
+          <width>800</width>
+          <height>800</height>
+          <format>R8G8B8</format>
+        </image>
+        <clip>
+          <near>0.02</near>
+          <far>300</far>
+        </clip>
+        <noise>
+          <type>gaussian</type>
+          <!-- Noise is sampled independently per pixel on each frame.
+               That pixel's noise value is added to each of its color
+               channels, which at that point lie in the range [0,1]. -->
+          <mean>0.0</mean>
+          <stddev>0.007</stddev>
+        </noise>
+      </camera>
+      <plugin name="camera_controller" filename="libgazebo_ros_camera.so">
+        <alwaysOn>true</alwaysOn>
+        <updateRate>0.0</updateRate>
+        <cameraName>teleop_cam</cameraName>
+        <imageTopicName>image_raw</imageTopicName>
+        <cameraInfoTopicName>camera_info</cameraInfoTopicName>
+        <frameName>camera_link</frameName>
+        <hackBaseline>0.07</hackBaseline>
+        <distortionK1>0.0</distortionK1>
+        <distortionK2>0.0</distortionK2>
+        <distortionK3>0.0</distortionK3>
+        <distortionT1>0.0</distortionT1>
+        <distortionT2>0.0</distortionT2>
+      </plugin>
+    </sensor>
+    </gazebo>
 </robot>

Commit message: updated files

File: src/gnc_description/urdf/gnc_robot.xacro (robot description, xacro)
@@ -28,8 +28,8 @@
     <xacro:arg name="use_nominal_extrinsics" default="True" />
     <xacro:realsense_d435 sensor_name="d435i" parent_link="base_link" rate="60.0">
-        <origin xyz="0.20 0 0.15" rpy="0 0 0"/>
+        <origin xyz="0.20 0 0.1805" rpy="0 0 0"/>
     </xacro:realsense_d435>
     <xacro:realsense_T265 sensor_name="t265" parent_link="base_link" rate="60.0">
-        <origin rpy="0 0 0" xyz="0 0 0.25"/>
+        <origin rpy="0 0 0" xyz="0 0 0.15"/>
     </xacro:realsense_T265>
     <!-- IMU GPS -->

Commit message: work on localization,planner,mapping, 50% finished

File: src/gnc_description/urdf/gnc_robot.xacro (robot description, xacro)
@@ -81,4 +81,16 @@
         </visual>
     </link>
+    <link name="magnetometer"/>
+    <gazebo>
+        <plugin name="GazeboRosMagnetic" filename="libhector_gazebo_ros_magnetic.so">
+	    <bodyName>magnetometer</bodyName>
+	    <topicName>/magnetometer/data</topicName>
+        </plugin>
+    </gazebo>
+    <joint name="mag_joint" type="fixed">
+        <origin xyz="-0.113 -0.0174 0.235" rpy="0 0 0"/>
+        <parent link="base_link"/>
+        <child link="magnetometer"/>
+    </joint>
     <gazebo reference="teleop_camera_link">
     <sensor type="camera" name="teleop_cam">

File: src/gnc_gazebo/sensors/_zedf9r.xacro (robot description, xacro)
@@ -36,5 +36,5 @@
         <gazebo>
             <plugin name="gps_controller" filename="libhector_gazebo_ros_gps.so">
-                <updateRate>30.0</updateRate>
+                <updateRate>10.0</updateRate>
                 <bodyName>${name}_link</bodyName>
                 <topicName>gps/fix</topicName>
@@ -46,5 +46,5 @@
                 <alwaysOn>true</alwaysOn>
                 <bodyName>${name}_link</bodyName>
-                <topicName>imu/data</topicName>
+                <topicName>imu/data_raw</topicName>
                 <serviceName>imu_service</serviceName>
                 <gaussianNoise>0.1</gaussianNoise>

Commit message: new commit

File: src/gnc_description/urdf/gnc_robot.xacro (robot description, xacro)
@@ -81,42 +81,17 @@
         </visual>
     </link>
-    <gazebo reference="teleop_camera_link">
-    <sensor type="camera" name="teleop_cam">
-      <update_rate>30.0</update_rate>
-      <camera name="teleop_cam">
-        <horizontal_fov>1.3962634</horizontal_fov>
-        <image>
-          <width>800</width>
-          <height>800</height>
-          <format>R8G8B8</format>
-        </image>
-        <clip>
-          <near>0.02</near>
-          <far>300</far>
-        </clip>
-        <noise>
-          <type>gaussian</type>
-          <!-- Noise is sampled independently per pixel on each frame.
-               That pixel's noise value is added to each of its color
-               channels, which at that point lie in the range [0,1]. -->
-          <mean>0.0</mean>
-          <stddev>0.007</stddev>
-        </noise>
-      </camera>
-      <plugin name="camera_controller" filename="libgazebo_ros_camera.so">
-        <alwaysOn>true</alwaysOn>
-        <updateRate>0.0</updateRate>
-        <cameraName>teleop_cam</cameraName>
-        <imageTopicName>image_raw</imageTopicName>
-        <cameraInfoTopicName>camera_info</cameraInfoTopicName>
-        <frameName>camera_link</frameName>
-        <hackBaseline>0.07</hackBaseline>
-        <distortionK1>0.0</distortionK1>
-        <distortionK2>0.0</distortionK2>
-        <distortionK3>0.0</distortionK3>
-        <distortionT1>0.0</distortionT1>
-        <distortionT2>0.0</distortionT2>
-      </plugin>
-    </sensor>
-    </gazebo>
+    <link name="base_to_shoulder_link"/>
+    <joint name="base_to_shoulder_joint" type="continuous">
+	<origin xyz="0 0 0" rpy="0 0 0"/>
+	<parent link="base_link"/>
+	<child link="base_to_shoulder_link"/>
+    </joint>
+<!--
+    <link name="shoulder_to_arm_link"/>
+-->
+<!--
+    <link name="teleop_camera_link"/>
+    <link name="teleop_camera_link"/>
+    <link name="teleop_camera_link"/>
+-->
 </robot>

Commit message: stack fully integrated, some bugs need fixing

File: src/gnc_description/urdf/gnc_robot.xacro (robot description, xacro)
@@ -24,7 +24,14 @@
     <xacro:wheel name="wheel_Left_Back" mass="${wheelMass}" parentLink="base_link" WheelXOrigin="${BackWheelYOrigin}" WheelYOrigin="${RightWheelXOrigin}"/>
     <!-- Camera -->
+    <!--
     <xacro:include filename="$(find gnc_gazebo)/sensors/_d435i.xacro" />
     <xacro:include filename="$(find gnc_gazebo)/sensors/_T265.xacro"/>
+    -->
+    <xacro:include filename="$(find gnc_gazebo)/sensors/_ZED.xacro"/>
     <xacro:arg name="use_nominal_extrinsics" default="True" />
+    <xacro:zed_camera name="ZEDMini" parent="base_link">
+        <origin xyz="0.20 0 0.1805" rpy="0 0 0"/>
+    </xacro:zed_camera>
+<!--
     <xacro:realsense_d435 sensor_name="d435i" parent_link="base_link" rate="60.0">
         <origin xyz="0.20 0 0.1805" rpy="0 0 0"/>
@@ -33,4 +40,5 @@
         <origin rpy="0 0 0" xyz="0 0 0.15"/>
     </xacro:realsense_T265>
+-->
     <!-- IMU GPS -->
     <xacro:include filename="$(find gnc_gazebo)/sensors/_zedf9r.xacro"/>

Commit message: after field test

File: src/gnc_description/urdf/gnc_robot.xacro (robot description, xacro)
@@ -27,5 +27,5 @@
     <xacro:include filename="$(find gnc_gazebo)/sensors/_ZED.xacro"/>
     <xacro:arg name="use_nominal_extrinsics" default="True" />
-    <xacro:zed_camera name="ZEDMini" parent="base_link">
+    <xacro:zed_camera name="zedm" parent="base_link">
         <origin xyz="0.0 0 0" rpy="0 0 0"/>
     </xacro:zed_camera>
@@ -40,5 +40,5 @@
     <!-- IMU GPS -->
     <xacro:include filename="$(find gnc_gazebo)/sensors/_zedf9r.xacro"/>
-    <xacro:Sparkfun_zedf9r name="zed_Sensor" parentLink="base_link">
+    <xacro:Sparkfun_zedf9r name="gps" parentLink="base_link">
        <origin rpy="0 0 0" xyz="0 0 0.15"/>
     </xacro:Sparkfun_zedf9r>

File: src/gnc_gazebo/sensors/_ZED.xacro (robot description, xacro)
@@ -3,5 +3,5 @@
     <xacro:macro name="zed_camera" params="name parent *origin">
         <!-- Physical properties -->
-        <link name="${name}">
+        <link name="${name}_base_link">
             <xacro:insert_block name="origin"/>
             <inertial>
@@ -23,11 +23,14 @@
                 </geometry>
             </collision>
-       </link>
+	</link>
+	<!--
         <link name="${name}_imu_link"></link>
+ -->
     	<joint name="${name}_${parent}_joint" type="fixed">
 		<parent link="${parent}"/>
-		<child link="${name}"/>
-		<origin xyz="0.6 0 0 " rpy="0 0 0 "/>
+		<child link="${name}_base_link"/>
+		<origin xyz="0.8 0 0 " rpy="0 0.785 0 "/>
 	</joint>
+	<!--
 	<joint name="${name}_imu_joint" type="fixed">
 		<parent link="${parent}"/>
@@ -46,4 +49,5 @@
 		<origin xyz="0 0 0" rpy="1.5708 3.142 1.5708"/>
 	</joint>
+	-->
         <!-- Stereo camera plugin for Gazebo -->
         <gazebo reference="${name}">

Commit message: zed2 migration

File: src/gnc_description/urdf/gnc_robot.xacro (robot description, xacro)
@@ -21,21 +21,14 @@
     <xacro:wheel name="wheel_Left_Back" mass="${wheelMass}" parentLink="base_link" WheelXOrigin="${BackWheelYOrigin}" WheelYOrigin="${RightWheelXOrigin}"/>
     <!-- Camera -->
-    <!--
-    <xacro:include filename="$(find gnc_gazebo)/sensors/_d435i.xacro" />
-    <xacro:include filename="$(find gnc_gazebo)/sensors/_T265.xacro"/>
-    -->
-    <xacro:include filename="$(find gnc_gazebo)/sensors/_ZED.xacro"/>
-    <xacro:arg name="use_nominal_extrinsics" default="True" />
-    <xacro:zed_camera name="zedm" parent="base_link">
-        <origin xyz="0.0 0 0" rpy="0 0 0"/>
-    </xacro:zed_camera>
-<!--
-    <xacro:realsense_d435 sensor_name="d435i" parent_link="base_link" rate="60.0">
-        <origin xyz="0.20 0 0.1805" rpy="0 0 0"/>
-    </xacro:realsense_d435>
-    <xacro:realsense_T265 sensor_name="t265" parent_link="base_link" rate="60.0">
-        <origin rpy="0 0 0" xyz="0 0 0.15"/>
-    </xacro:realsense_T265>
--->
+    <xacro:macro name="gnc_robot_sim" params="robot_ns:='${robot_ns}'">
+	    <xacro:zed2_gazebo robot_ns="${robot_ns}"/>
+    </xacro:macro>
+    <xacro:include filename="$(find gnc_gazebo)/sensors/_ZED2.xacro"/>
+    <xacro:zed2 link_prefix="" joint_prefix="" />
+    <joint name="zed2_camera_center_joint" type="fixed">
+      <parent link="base_link"/>
+      <child link="zed2_camera_center"/>
+      <origin xyz="0.6 0 0.0486" rpy="0 0.12637657 0"/>
+    </joint>
     <!-- IMU GPS -->
     <xacro:include filename="$(find gnc_gazebo)/sensors/_zedf9r.xacro"/>
@@ -43,5 +36,4 @@
        <origin rpy="0 0 0" xyz="0 0 0.15"/>
     </xacro:Sparkfun_zedf9r>
-    <!-- Gazebo code for protobot -->
     <gazebo>
         <plugin filename="libgazebo_ros_control.so" name="gazebo_ros_control">
@@ -66,21 +58,9 @@
     </gazebo>
     <joint name="teleop_camera_joint" type="fixed">
-    <origin xyz="-0.181 0.19 0.695" rpy="0 0 0"/>
-    <parent link="base_link"/>
-    <child link="teleop_camera_link"/>
+	<origin xyz="-0.181 0.19 0.695" rpy="0 0 0"/>
+    	<parent link="base_link"/>
+    	<child link="teleop_camera_link"/>
     </joint>
     <link name="teleop_camera_link"/>
-    <link name="magnetometer"/>
-    <gazebo>
-        <plugin name="GazeboRosMagnetic" filename="libhector_gazebo_ros_magnetic.so">
-	    <bodyName>magnetometer</bodyName>
-	    <topicName>/magnetometer/data</topicName>
-        </plugin>
-    </gazebo>
-    <joint name="mag_joint" type="fixed">
-        <origin xyz="-0.113 -0.0174 0.235" rpy="0 0 0"/>
-        <parent link="base_link"/>
-        <child link="magnetometer"/>
-    </joint>
     <gazebo reference="teleop_camera_link">
     <sensor type="camera" name="teleop_cam">

File: src/gnc_gazebo/sensors/_zedf9r.xacro (robot description, xacro)
@@ -42,5 +42,6 @@
                 <gaussianNoise>2</gaussianNoise>
                 <alwayson>true</alwayson>
-            </plugin>
+	</plugin>
+	<!--
             <plugin name="imu_plugin" filename="libgazebo_ros_imu.so">
                 <alwaysOn>true</alwaysOn>
@@ -50,5 +51,6 @@
                 <gaussianNoise>0.1</gaussianNoise>
                 <updateRate>30.0</updateRate>
-            </plugin>
+		</plugin>
+	-->
         </gazebo>
     </xacro:macro>

Commit message: autonav almost done

File: src/gnc_description/urdf/gnc_robot.xacro (robot description, xacro)
@@ -24,10 +24,13 @@
 	    <xacro:zed2_gazebo robot_ns="${robot_ns}"/>
     </xacro:macro>
+    <!--
     <xacro:include filename="$(find gnc_gazebo)/sensors/_ZED2.xacro"/>
     <xacro:zed2 link_prefix="" joint_prefix="" />
+	    -->
+    <link name="zed2_base_link"/>
     <joint name="zed2_camera_center_joint" type="fixed">
       <parent link="base_link"/>
-      <child link="zed2_camera_center"/>
-      <origin xyz="0.6 0 0.0486" rpy="0 0.12637657 0"/>
+      <child link="zed2_base_link"/>
+      <origin xyz="0.6 0 0.0486" rpy="0 0.2782 0"/>
     </joint>
     <!-- IMU GPS -->

Commit message: work

File: src/gnc_description/urdf/gnc_robot.xacro (robot description, xacro)
@@ -24,8 +24,12 @@
 	    <xacro:zed2_gazebo robot_ns="${robot_ns}"/>
     </xacro:macro>
-    <!--
     <xacro:include filename="$(find gnc_gazebo)/sensors/_ZED2.xacro"/>
     <xacro:zed2 link_prefix="" joint_prefix="" />
-	    -->
+    <joint name="zed2_camera_center_joint" type="fixed">
+    	<parent link='base_link'/>
+	<child link="zed2_camera_center"/>
+	<origin xyz="0.6 0 0.0486" rpy="0 0.2782 0"/>
+    </joint>
+    <!--
     <link name="zed2_base_link"/>
     <joint name="zed2_camera_center_joint" type="fixed">
@@ -34,4 +38,5 @@
       <origin xyz="0.6 0 0.0486" rpy="0 0.2782 0"/>
     </joint>
+    -->
     <!-- IMU GPS -->
     <xacro:include filename="$(find gnc_gazebo)/sensors/_zedf9r.xacro"/>

File: src/gnc_gazebo/sensors/_ZED2.xacro (robot description, xacro)
@@ -124,5 +124,5 @@
         </camera>
         <plugin name="camera_controller" filename="libgazebo_ros_camera.so">
-          <cameraName>zed2/left_raw</cameraName>
+		<cameraName>zed2/zed_node/left_raw</cameraName>
           <imageTopicName>image_raw_color</imageTopicName>
           <cameraInfoTopicName>camera_info</cameraInfoTopicName>
@@ -163,9 +163,9 @@
         <plugin name="camera_controller" filename="libgazebo_ros_openni_kinect.so">
           <cameraName>zed2</cameraName>
-          <imageTopicName>left/image_rect_color</imageTopicName>
-          <cameraInfoTopicName>left/camera_info</cameraInfoTopicName>
-          <depthImageTopicName>depth/depth_registered</depthImageTopicName>
-          <depthImageInfoTopicName>depth/camera_info</depthImageInfoTopicName>
-          <pointCloudTopicName>point_cloud/cloud_registered</pointCloudTopicName>
+	  <imageTopicName>zed_node/left/image_rect_color</imageTopicName>
+	  <cameraInfoTopicName>zed_node/left/camera_info</cameraInfoTopicName>
+	  <depthImageTopicName>zed_node/depth/depth_registered</depthImageTopicName>
+	  <depthImageInfoTopicName>zed_node/depth/camera_info</depthImageInfoTopicName>
+	  <pointCloudTopicName>zed_node/point_cloud/cloud_registered</pointCloudTopicName>
           <pointCloudCutoff>0.3</pointCloudCutoff>
           <pointCloudCutoffMax>20.0</pointCloudCutoffMax>
@@ -212,5 +212,5 @@
         </camera>
         <plugin name="camera_controller" filename="libgazebo_ros_camera.so">
-          <cameraName>zed2/right_raw</cameraName>
+		<cameraName>zed2/zed_node/right_raw</cameraName>
           <imageTopicName>image_raw_color</imageTopicName>
           <cameraInfoTopicName>camera_info</cameraInfoTopicName>
@@ -250,5 +250,5 @@
         </camera>
         <plugin name="camera_controller" filename="libgazebo_ros_camera.so">
-          <cameraName>zed2/right</cameraName>
+		<cameraName>zed2/zed_node/right</cameraName>
           <imageTopicName>image_rect_color</imageTopicName>
           <cameraInfoTopicName>camera_info</cameraInfoTopicName>
@@ -266,5 +266,5 @@
         <update_rate>100</update_rate>
         <plugin filename="libgazebo_ros_imu_sensor.so" name="imu_plugin">
-          <topicName>zed2/imu/data</topicName>
+		<topicName>zed2/zed_node/imu/data</topicName>
           <frameName>zed2_imu_link</frameName>
           <updateRateHZ>100.0</updateRateHZ>
@@ -282,5 +282,5 @@
 		<updateRate>50</updateRate>
                 <bodyName>zed2_camera_center</bodyName>
-		<topicName>zed2/odom/sample</topicName>
+		<topicName>zed2/zed_node/odom</topicName>
                 <gaussianNoise>0.001</gaussianNoise>
                 <frameName>world</frameName>
