Commit message: mdrs world working

File: src/gnc_gazebo/sensors/_T265.xacro (robot description, xacro)
@@ -92,5 +92,5 @@
             <origin rpy="1.57 0 1.57" xyz="0 0 0"/>
             <geometry>
-                <mesh filename="package://gnc_gazebo/meshes/realsense_t265.stl" scale="0.001 0.001 0.001"/>
+                <mesh filename="package://gnc_gazebo/mesh/realsense_t265.stl" scale="0.001 0.001 0.001"/>
             </geometry>
         </visual>

File: src/gnc_gazebo/sensors/_d435i.xacro (robot description, xacro)
@@ -44,5 +44,5 @@
         <origin xyz="${d435_cam_mount_from_center_offset} ${-d435_cam_depth_py} 0" rpy="${pi/2} 0 ${pi/2}"/>
         <geometry>
-          <mesh filename="package://gnc_gazebo/meshes/d435.dae" />
+          <mesh filename="package://gnc_gazebo/mesh/d435.dae" />
         </geometry>
       </visual>
